File: SB-4S5A.kicad_pcb (KiCad board)
At the start: 4 copper layers, 100 x 50 mm, 41 parts, among them J1 CONN_01X06, Q1 CSD17308Q3, Q2 CSD17308Q3, Q3 2N7002, U1 bq40z50-r2

Commit message: Almost done, can't freaking decide on a connector...
Parts:
- J1: value CONN_01X06 -> Conn_02x03_Top_Bottom; footprint TI SBS:14110613002XXX -> Connectors_Molex:Molex_Microfit3_Header_02x03_Angled_43045-060x
- moved R18 18.8 mm to (93.0, 87.2), turned to 180 degrees
- moved R17 17.5 mm to (93.0, 86.0), turned to 180 degrees
- moved R20 16.3 mm to (93.0, 84.8), turned to 180 degrees
- moved R19 15.2 mm to (93.0, 83.5), turned to 180 degrees
- moved J1 5.22 mm to (89.8, 69.1)
- moved C1 4.85 mm to (101.2, 77.5)
- moved C2 4.85 mm to (99.2, 77.5)
- moved C3 4.85 mm to (97.1, 77.5)
- moved C4 4.85 mm to (95.0, 77.5)
- moved D1 4.85 mm to (102.2, 75.5)
- moved R2 4.85 mm to (100.0, 76.0)
- moved R3 4.85 mm to (98.8, 76.0)
- moved R4 4.85 mm to (97.5, 76.0)
- moved R5 4.85 mm to (96.2, 76.0)
- moved C5 4.00 mm to (91.2, 77.0)
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Connections:
- J1 pad 1: /BTP_INT -> PACK+
- J1 pad 2: /~PRES~ -> PACK-
- J1 pad 3: /SMBD -> /SMBC
- J1 pad 4: /SMBC -> /SMBD
- J1 pad 5: PACK- -> /~PRES~
- J1 pad 6: PACK+ -> /BTP_INT
Routing:
- net /BAT+: track 31.7 -> 2.50 mm, vias 2 -> 1
- net /BTP_INT_: track 24.0 -> 3.03 mm, vias 2 -> 0
- net /~PRES/SHDN~_: track 23.9 -> 3.49 mm, vias 2 -> 0
- net /SMBD_: track 24.1 -> 4.70 mm, vias 2 -> 0
- net /SMBC_: track 24.9 -> 5.79 mm, vias 2 -> 0
- net /VC1A: track 19.4 -> 7.42 mm
- net /VC4: track 14.2 -> 6.56 mm
- net /VC3: track 12.8 -> 5.24 mm
- net /VC2: track 10.8 -> 4.64 mm
- net /SMBC: track 5.40 -> 0.00 mm
- net /BAT: track 13.1 -> 8.02 mm
- net /BTP_INT: track 4.92 -> 0.00 mm
- net /VC1: track 9.76 -> 5.15 mm
- net /~PRES~: track 4.44 -> 0.10 mm
- net /SMBD: track 4.31 -> 0.10 mm
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
Commit message: Ready to send to manufacturer.
Parts:
- added REF**: MountingHole_3.2mm_M3_Pad, Mounting_Holes:MountingHole_3.2mm_M3_Pad, F.Cu at (75.0, 65.0)
- J1: value Conn_02x03_Top_Bottom -> LEMO6; footprint Connectors_Molex:Molex_Microfit3_Header_02x03_Angled_43045-060x -> Connectors_Samtec:SL-106-X-XX_1x06
- moved BT1 10.0 mm to (95.0, 100.0)
- moved BT2 10.0 mm to (145.0, 100.0)
- moved BT3 10.0 mm to (145.0, 100.0)
- moved BT4 10.0 mm to (95.0, 100.0)
- moved C1 10.0 mm to (101.2, 87.5)
- moved C2 10.0 mm to (99.2, 87.5)
- moved C3 10.0 mm to (97.1, 87.5)
- moved C4 10.0 mm to (95.0, 87.5)
- moved C5 10.0 mm to (91.2, 87.0)
- moved C6 10.0 mm to (101.8, 89.8)
- moved D1 10.0 mm to (102.2, 85.5)
- moved Q1 10.0 mm to (73.8, 85.0)
- moved Q2 10.0 mm to (73.7, 80.0)
- moved Q3 10.0 mm to (72.8, 74.5)
- moved R1 10.0 mm to (89.0, 95.0)
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Connections:
- U1 pad 17: Net-(U1-Pad17) -> (no net)
- U1 pad 20: Net-(U1-Pad20) -> (no net)
- U1 pad 21: Net-(U1-Pad21) -> (no net)
- U1 pad 22: Net-(U1-Pad22) -> (no net)
- U1 pad 25: Net-(U1-Pad25) -> (no net)
- U1 pad 30: Net-(U1-Pad30) -> (no net)
Routing:
- net /BAT+: track 2.50 -> 29.5 mm, vias 1 -> 2
- net /BTP_INT: track 0.00 -> 24.4 mm, vias 0 -> 1
- net /SMBC: track 0.00 -> 24.2 mm, vias 0 -> 1
- net /~PRES~: track 0.10 -> 23.9 mm, vias 0 -> 1
- net /SMBD: track 0.10 -> 23.3 mm, vias 0 -> 1
- net /VC1A: track 7.42 -> 16.2 mm
- net /VC2A: track 62.9 -> 70.8 mm
- net /VC3A: track 16.7 -> 24.2 mm

Commit message: Fix FUSE pin floating.
Connections:
- U1 pad 25: (no net) -> GNDD
Changed lines of the file:
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@@
   (page A4)
   (layers
-    (0 F.Cu signal hide)
+    (0 F.Cu signal)
     (1 In1.Cu mixed hide)
     (2 In2.Cu mixed hide)
@@
     (pad 24 smd oval (at 1.9 -1.4) (size 0.2 0.6) (layers F.Cu F.Paste F.Mask)
       (net 1 GNDD))
-    (pad 25 smd oval (at 1.4 -1.9 270) (size 0.2 0.6) (layers F.Cu F.Paste F.Mask))
+    (pad 25 smd oval (at 1.4 -1.9 270) (size 0.2 0.6) (layers F.Cu F.Paste F.Mask)
+      (net 1 GNDD))
     (pad 26 smd oval (at 1 -1.9 270) (size 0.2 0.6) (layers F.Cu F.Paste F.Mask)
       (net 30 /_VCC_))
@@
   (segment (start 103.3 85.925) (end 103.3 85.5) (width 0.2) (layer F.Cu) (net 21) (status 20))
   (segment (start 91.2 95.4) (end 91.8 96) (width 0.2) (layer F.Cu) (net 22))
-  (segment (start 91.8 96) (end 92.55 96) (width 0.2) (layer F.Cu) (net 22))
+  (segment (start 91.8 96) (end 92.55 96) (width 0.2) (layer F.Cu) (net 22) (status 20))
   (segment (start 91.2 94.4) (end 91.2 95.4) (width 0.2) (layer F.Cu) (net 22))
   (segment (start 90.45 93.65) (end 91.2 94.4) (width 0.2) (layer F.Cu) (net 22))
   (segment (start 90.45 89) (end 90.45 93.65) (width 0.2) (layer F.Cu) (net 22))
-  (segment (start 92.62 75) (end 90.45 77.17) (width 0.2) (layer In2.Cu) (net 22))
+  (segment (start 92.62 75) (end 90.45 77.17) (width 0.2) (layer In2.Cu) (net 22) (status 10))
   (segment (start 90.45 77.17) (end 90.45 89) (width 0.2) (layer In2.Cu) (net 22))
   (via (at 90.45 89) (size 0.8) (drill 0.4) (layers F.Cu B.Cu) (net 22))
@@
   (segment (start 90.08 88.42) (end 89.5 89) (width 0.2) (layer In2.Cu) (net 23))
   (segment (start 91.1 93.8) (end 92.05 94.75) (width 0.2) (layer F.Cu) (net 24))
-  (segment (start 92.05 94.75) (end 92.55 94.75) (width 0.2) (layer F.Cu) (net 24))
+  (segment (start 92.05 94.75) (end 92.55 94.75) (width 0.2) (layer F.Cu) (net 24) (status 20))
   (segment (start 91.1 89.7) (end 91.1 93.8) (width 0.2) (layer F.Cu) (net 24))
   (segment (start 90.8 88.4) (end 91.1 88.7) (width 0.2) (layer In2.Cu) (net 24))
@@
   (segment (start 91.2 76.95) (end 90.8 77.35) (width 0.2) (layer In2.Cu) (net 24))
   (segment (start 93.21 76.95) (end 91.2 76.95) (width 0.2) (layer In2.Cu) (net 24))
-  (segment (start 95.16 75) (end 93.21 76.95) (width 0.2) (layer In2.Cu) (net 24))
+  (segment (start 95.16 75) (end 93.21 76.95) (width 0.2) (layer In2.Cu) (net 24) (status 10))
   (segment (start 92.55 94.75) (end 92.55 94.65) (width 0.2) (layer F.Cu) (net 24) (status 30))
   (segment (start 91.75 90.4) (end 91.75 93.1) (width 0.2) (layer F.Cu) (net 25))
   (segment (start 91.75 93.1) (end 92.15 93.5) (width 0.2) (layer F.Cu) (net 25))
-  (segment (start 92.15 93.5) (end 92.55 93.5) (width 0.2) (layer F.Cu) (net 25))
+  (segment (start 92.15 93.5) (end 92.55 93.5) (width 0.2) (layer F.Cu) (net 25) (status 20))
   (segment (start 91.15 88.25) (end 91.75 88.85) (width 0.2) (layer In2.Cu) (net 25))
   (segment (start 91.75 88.85) (end 91.75 90.4) (width 0.2) (layer In2.Cu) (net 25))
@@
   (segment (start 91.35 77.3) (end 91.15 77.5) (width 0.2) (layer In2.Cu) (net 25))
   (segment (start 95.4 77.3) (end 91.35 77.3) (width 0.2) (layer In2.Cu) (net 25))
-  (segment (start 97.7 75) (end 95.4 77.3) (width 0.2) (layer In2.Cu) (net 25))
+  (segment (start 97.7 75) (end 95.4 77.3) (width 0.2) (layer In2.Cu) (net 25) (status 10))
   (segment (start 77.3 86) (end 77.3 84.75) (width 0.2) (layer F.Cu) (net 27) (status 30))
   (segment (start 77.3 84.75) (end 77.25 84.7) (width 0.2) (layer F.Cu) (net 27) (status 30))
