File: SB-4S5A.sch (KiCad schematic (older format))
At the start: 39 parts, among them J1 I2C, J2 BATIO, Q1 CSD19537Q3, Q2 CSD19537Q3, Q3 2N7002, U1 bq40z50-r2

Commit message: Some updates, net-ties and such.
Parts:
- removed Q1, Q2: CSD19537Q3, Housings_SON:VSON-8_3.3x3.3mm_Pitch0.65mm_NexFET, symbol CSD19537Q3
- added Q1, Q2: CSD17308Q3, Housings_SON:VSON-8_3.3x3.3mm_Pitch0.65mm_NexFET, symbol CSD19534Q5A
Changed lines of the file:
@@
 $EndComp
 $Comp
-L GND #PWR01
+L GND #PWR1
 U 1 1 597D5EFB
 P 1550 5350
-F 0 "#PWR01" H 1550 5100 50  0001 C CNN
+F 0 "#PWR1" H 1550 5100 50  0001 C CNN
 F 1 "GND" H 1550 5200 50  0000 C CNN
 F 2 "" H 1550 5350 50  0001 C CNN
@@
 $EndComp
 $Comp
-L GNDD #PWR02
+L GNDD #PWR2
 U 1 1 597D5F72
 P 2100 5350
-F 0 "#PWR02" H 2100 5100 50  0001 C CNN
+F 0 "#PWR2" H 2100 5100 50  0001 C CNN
 F 1 "GNDD" H 2100 5200 50  0000 C CNN
 F 2 "" H 2100 5350 50  0001 C CNN
@@
 	1    2100 5350
 	1    0    0    -1
-$EndComp
-$Comp
-L CSD19537Q3 Q1
-U 1 1 597D6A2B
-P 5550 1550
-F 0 "Q1" H 5550 1967 50  0000 C CNN
-F 1 "CSD19537Q3" H 5550 1876 50  0000 C CNN
-F 2 "Housings_SON:VSON-8_3.3x3.3mm_Pitch0.65mm_NexFET" H 5350 1200 50  0001 L CIN
-F 3 "" H 5350 1850 50  0000 L CNN
-	1    5550 1550
-	1    0    0    -1
-$EndComp
-$Comp
-L CSD19537Q3 Q2
-U 1 1 597D6D1F
-P 6550 1550
-F 0 "Q2" H 6550 1967 50  0000 C CNN
-F 1 "CSD19537Q3" H 6550 1876 50  0000 C CNN
-F 2 "Housings_SON:VSON-8_3.3x3.3mm_Pitch0.65mm_NexFET" H 6350 1200 50  0001 L CIN
-F 3 "" H 6350 1850 50  0000 L CNN
-	1    6550 1550
-	-1   0    0    -1
 $EndComp
 $Comp
@@
 $EndComp
 $Comp
-L GNDD #PWR03
+L GNDD #PWR7
 U 1 1 597D870F
 P 6650 4650
-F 0 "#PWR03" H 6650 4400 50  0001 C CNN
+F 0 "#PWR7" H 6650 4400 50  0001 C CNN
 F 1 "GNDD" H 6650 4500 50  0000 C CNN
 F 2 "" H 6650 4650 50  0001 C CNN
@@
 NoConn ~ 6550 3700
 $Comp
-L GNDD #PWR04
+L GNDD #PWR5
 U 1 1 597D8929
 P 5450 4650
-F 0 "#PWR04" H 5450 4400 50  0001 C CNN
+F 0 "#PWR5" H 5450 4400 50  0001 C CNN
 F 1 "GNDD" H 5450 4500 50  0000 C CNN
 F 2 "" H 5450 4650 50  0001 C CNN
@@
 $EndComp
 $Comp
-L GNDD #PWR05
+L GNDD #PWR6
 U 1 1 597D8A8D
 P 6650 3400
-F 0 "#PWR05" H 6650 3150 50  0001 C CNN
+F 0 "#PWR6" H 6650 3150 50  0001 C CNN
 F 1 "GNDD" H 6650 3250 50  0000 C CNN
 F 2 "" H 6650 3400 50  0001 C CNN
@@
 Connection ~ 3750 4500
 $Comp
-L GNDD #PWR06
+L GNDD #PWR4
 U 1 1 597DD005
 P 4500 4800
-F 0 "#PWR06" H 4500 4550 50  0001 C CNN
+F 0 "#PWR4" H 4500 4550 50  0001 C CNN
 F 1 "GNDD" H 4500 4650 50  0000 C CNN
 F 2 "" H 4500 4800 50  0001 C CNN
@@
 Connection ~ 9050 4850
 $Comp
-L GNDS #PWR07
+L GNDS #PWR3
 U 1 1 597DE8AD
 P 4250 5300
-F 0 "#PWR07" H 4250 5050 50  0001 C CNN
+F 0 "#PWR3" H 4250 5050 50  0001 C CNN
 F 1 "GNDS" H 4255 5127 50  0000 C CNN
 F 2 "" H 4250 5300 50  0001 C CNN
@@
 Connection ~ 3850 5100
 $Comp
-L GNDS #PWR08
+L GNDS #PWR9
 U 1 1 597DEA01
 P 9050 5350
-F 0 "#PWR08" H 9050 5100 50  0001 C CNN
+F 0 "#PWR9" H 9050 5100 50  0001 C CNN
 F 1 "GNDS" H 9055 5177 50  0000 C CNN
 F 2 "" H 9050 5350 50  0001 C CNN
@@
 	7700 1750 7800 1750
 $Comp
-L GNDS #PWR09
+L GNDS #PWR8
 U 1 1 597E029E
 P 7800 2250
-F 0 "#PWR09" H 7800 2000 50  0001 C CNN
+F 0 "#PWR8" H 7800 2000 50  0001 C CNN
 F 1 "GNDS" H 7805 2077 50  0000 C CNN
 F 2 "" H 7800 2250 50  0001 C CNN
@@
 Wire Wire Line
 	4250 5250 4250 5300
+$Comp
+L CSD19534Q5A Q1
+U 1 1 597E6AFE
+P 5550 1550
+F 0 "Q1" H 5550 1967 50  0000 C CNN
+F 1 "CSD17308Q3" H 5550 1876 50  0000 C CNN
+F 2 "Housings_SON:VSON-8_3.3x3.3mm_Pitch0.65mm_NexFET" H 5550 1750 50  0001 C CIN
+F 3 "" V 5550 1550 50  0001 L CNN
+	1    5550 1550
+	1    0    0    -1
+$EndComp
+$Comp
+L CSD19534Q5A Q2
+U 1 1 597E6C1E
+P 6550 1550
+F 0 "Q2" H 6550 1967 50  0000 C CNN
+F 1 "CSD17308Q3" H 6550 1876 50  0000 C CNN
+F 2 "Housings_SON:VSON-8_3.3x3.3mm_Pitch0.65mm_NexFET" H 6550 1750 50  0001 C CIN
+F 3 "" V 6550 1550 50  0001 L CNN
+	1    6550 1550
+	-1   0    0    -1
+$EndComp
 $EndSCHEMATC

Commit message: Added battery footprint
Parts:
- BT1: renamed from BT4; footprint (none) -> TI SBS:105070
- BT2: renamed from BT3; footprint (none) -> TI SBS:105070
- BT3: renamed from BT2; footprint (none) -> TI SBS:105070
- BT4: renamed from BT1; footprint (none) -> TI SBS:105070
- renumbered C1 to C?, C2 to C?, C3 to C?, C4 to C?, C5 to C?, C6 to C?, D1 to D?, J1 to J?, J2 to J?, Q3 to Q?, Q1 to Q?, Q2 to Q?, R8 to R?, R11 to R?, R10 to R?, R16 to R?, R15 to R?, R1 to R?, R2 to R?, R3 to R?, R4 to R?, R6 to R?, R5 to R?, R7 to R?, R9 to R?, R12 to R?, R13 to R?, R14 to R?, R17 to R?, R18 to R?, TH1 to TH?, TH2 to TH?, TH3 to TH?, TH4 to TH?, U1 to U?

Commit message: Reannotate
Parts:
- gave numbers to parts that had none: 35
- renumbered BT4 to BT1, BT3 to BT2, BT2 to BT3, BT1 to BT4

Commit message: Finish place and routing.
Parts:
- removed J1: I2C, Connectors:Grove_1x04, symbol CONN_01X04
- removed J2: BATIO, Connectors:Grove_1x04, symbol CONN_01X04
- removed R9: NET-TIE, Oddities:NetTie-I_Connected, symbol R
- added J1: CONN_01X06, TI SBS:14110613002XXX, symbol CONN_01X06
- added R19, R20: 100R, Resistors_SMD:R_0402, symbol R
Connections:
- net labels added: BAT, BAT+, BAT-, BTP_INT, BTP_INT_, CHG, CHG_G, DSG, DSG_G, MID, PACK, PBI, SMBC, SMBC_, SMBD, SMBD_, SRN, SRP, VC1, VC1A, VC2, VC2A, VC3, VC3A, VC4, _VCC_, ~PRES/SHDN~_, ~PRES~
- net labels removed: GND, GNDS
- wire segments 129 -> 139
- no-connect marks 8 -> 6
Other:
- moved on the sheet: D1, Q3, R15, R16, R17, R18

Commit message: Convert to "KiCad 5.0" format.
Other stuff
Parts:
- BT1, BT2, BT3, BT4: symbol Battery_Cell -> device:Battery_Cell
- C1, C2, C3, C4, C5, C6: symbol C -> device:C
- D1: symbol D_Schottky -> device:D_Schottky
- J1: symbol CONN_01X06 -> Connector:Conn_01x06
- Q1, Q2: symbol CSD19534Q5A -> SB-4S5A-rescue:CSD19534Q5A-RESCUE-SB-4S5A
- Q3: symbol 2N7002 -> Transistor:2N7002
- R1, R10, R11, R12, R13, R14, R15, R16, R18, R2, R20, R3, R4, R5, R6, R7, R8: symbol R -> SB-4S5A-rescue:R-RESCUE-SB-4S5A
- R17, R19: symbol R -> device:R
- TH1, TH2, TH3, TH4: symbol Thermistor_NTC -> device:Thermistor_NTC
- U1: symbol bq40z50-r2 -> SB-4S5A-rescue:bq40z50-r2-RESCUE-SB-4S5A
Changed lines of the file:
@@
-EESchema Schematic File Version 2
-LIBS:power
-LIBS:device
-LIBS:transistors
-LIBS:conn
-LIBS:linear
-LIBS:regul
-LIBS:74xx
-LIBS:cmos4000
-LIBS:adc-dac
-LIBS:memory
-LIBS:xilinx
-LIBS:microcontrollers
-LIBS:dsp
-LIBS:microchip
-LIBS:analog_switches
-LIBS:motorola
-LIBS:texas
-LIBS:intel
-LIBS:audio
-LIBS:interface
-LIBS:digital-audio
-LIBS:philips
-LIBS:display
-LIBS:cypress
-LIBS:siliconi
-LIBS:opto
-LIBS:atmel
-LIBS:contrib
-LIBS:valves
-LIBS:ti-sbs
+EESchema Schematic File Version 4
 LIBS:SB-4S5A-cache
 EELAYER 26 0
@@
 $EndDescr
 $Comp
-L bq40z50-r2 U1
+L SB-4S5A-rescue:bq40z50-r2-RESCUE-SB-4S5A U1
 U 1 1 597C0F06
 P 6050 3850
@@
 $EndComp
 $Comp
-L Battery_Cell BT1
+L device:Battery_Cell BT1
 U 1 1 597D5B15
 P 1650 3000
@@
 $EndComp
 $Comp
-L Battery_Cell BT2
+L device:Battery_Cell BT2
 U 1 1 597D5BA3
 P 1650 3500
@@
 $EndComp
 $Comp
-L Battery_Cell BT3
+L device:Battery_Cell BT3
 U 1 1 597D5BC7
 P 1650 4000
@@
 $EndComp
 $Comp
-L Battery_Cell BT4
+L device:Battery_Cell BT4
 U 1 1 597D5C07
 P 1650 4500
@@
 $EndComp
 $Comp
-L GNDD #PWR02
+L power:GNDD #PWR02
 U 1 1 597D5F72
 P 2100 5350
@@
 $EndComp
 $Comp
-L R R10
+L SB-4S5A-rescue:R-RESCUE-SB-4S5A R10
 U 1 1 597D7CD3
 P 5050 1500
@@
 $EndComp
 $Comp
-L R R13
+L SB-4S5A-rescue:R-RESCUE-SB-4S5A R13
 U 1 1 597D7E73
 P 7050 1500
@@
 $EndComp
 $Comp
-L D_Schottky D1
+L device:D_Schottky D1
 U 1 1 597D8090
 P 5150 3200
@@
 $EndComp
 $Comp
-L R R12
+L SB-4S5A-rescue:R-RESCUE-SB-4S5A R12
 U 1 1 597D81DC
 P 6050 2300
@@
 $EndComp
 $Comp
-L GNDD #PWR07
+L power:GNDD #PWR07
 U 1 1 597D870F
 P 6650 4650
@@
 NoConn ~ 6550 3700
 $Comp
-L GNDD #PWR05
+L power:GNDD #PWR05
 U 1 1 597D8929
 P 5450 4650
@@
 $EndComp
 $Comp
-L GNDD #PWR06
+L power:GNDD #PWR06
 U 1 1 597D8A8D
 P 6650 3400
@@
 $EndComp
 $Comp
-L R R18
+L SB-4S5A-rescue:R-RESCUE-SB-4S5A R18
 U 1 1 597D9352
 P 8600 4300
@@
 $EndComp
 $Comp
-L R R17
+L device:R R17
 U 1 1 597D94E6
 P 8350 4400
@@
 $EndComp
 $Comp
-L R R2
+L SB-4S5A-rescue:R-RESCUE-SB-4S5A R2
 U 1 1 597D97AB
 P 2250 2700
@@
 $EndComp
 $Comp
-L R R3
+L SB-4S5A-rescue:R-RESCUE-SB-4S5A R3
 U 1 1 597D983F
 P 2250 3200
@@
 $EndComp
 $Comp
-L R R4
+L SB-4S5A-rescue:R-RESCUE-SB-4S5A R4
 U 1 1 597D9881
 P 2250 3700
@@
 $EndComp
 $Comp
-L R R5
+L SB-4S5A-rescue:R-RESCUE-SB-4S5A R5
 U 1 1 597D98C3
 P 2250 4200
@@
 $EndComp
 $Comp
-L C C1
+L device:C C1
 U 1 1 597DA829
 P 2650 2950
@@
 $EndComp
 $Comp
-L C C2
+L device:C C2
 U 1 1 597DA9C3
 P 2650 3450
@@
 $EndComp
 $Comp
-L C C3
+L device:C C3
 U 1 1 597DAA35
 P 2650 3950
@@
 $EndComp
 $Comp
-L C C4
+L device:C C4
 U 1 1 597DAA98
 P 2650 4450
@@
 $EndComp
 $Comp
-L Thermistor_NTC TH1
+L device:Thermistor_NTC TH1
 U 1 1 597DB329
 P 4500 4450
@@
 $EndComp
 $Comp
-L Thermistor_NTC TH2
+L device:Thermistor_NTC TH2
 U 1 1 597DB805
 P 4650 4450
@@
 $EndComp
 $Comp
-L Thermistor_NTC TH3
+L device:Thermistor_NTC TH3
 U 1 1 597DB855
 P 4800 4450
@@
 $EndComp
 $Comp
-L Thermistor_NTC TH4
+L device:Thermistor_NTC TH4
 U 1 1 597DB899
 P 4950 4450
@@
 $EndComp
 $Comp
-L R R7
+L SB-4S5A-rescue:R-RESCUE-SB-4S5A R7
 U 1 1 597DBE1F
 P 3500 5100
@@
 $EndComp
 $Comp
-L R R6
+L SB-4S5A-rescue:R-RESCUE-SB-4S5A R6
 U 1 1 597DC663
 P 3250 4750
@@
 $EndComp
 $Comp
-L R R8
+L SB-4S5A-rescue:R-RESCUE-SB-4S5A R8
 U 1 1 597DC787
 P 3750 4750
@@
 $EndComp
 $Comp
-L C C5
+L device:C C5
 U 1 1 597DC7E1
 P 3500 4500
@@
 Connection ~ 3750 4500
 $Comp
-L GNDD #PWR04
+L power:GNDD #PWR04
 U 1 1 597DD005
 P 4500 4800
@@
 	5250 3650 5250 5000
 $Comp
-L R R11
+L SB-4S5A-rescue:R-RESCUE-SB-4S5A R11
 U 1 1 597DEEA7
 P 5050 2300
@@
 $EndComp
 $Comp
-L 2N7002 Q3
+L Transistor:2N7002 Q3
 U 1 1 597DF192
 P 7350 1750
@@
 	7250 2050 7050 2050
 $Comp
-L R R14
+L SB-4S5A-rescue:R-RESCUE-SB-4S5A R14
 U 1 1 597DF55A
 P 7050 2300
@@
 Connection ~ 7050 2050
 $Comp
-L R R15
+L SB-4S5A-rescue:R-RESCUE-SB-4S5A R15
 U 1 1 597E00A9
 P 7650 2000
@@
 	7650 1750 7650 1850
 $Comp
-L R R16
+L SB-4S5A-rescue:R-RESCUE-SB-4S5A R16
 U 1 1 597E0ADE
 P 7900 2000
@@
 Connection ~ 7900 1350
 $Comp
-L C C6
+L device:C C6
 U 1 1 597E0DFB
 P 4250 4450
@@
 Connection ~ 7050 1350
 $Comp
-L R R1
+L SB-4S5A-rescue:R-RESCUE-SB-4S5A R1
 U 1 1 597E22A7
 P 1900 5300
@@
 	2100 5300 2100 5350
 $Comp
-L CSD19534Q5A Q1
+L SB-4S5A-rescue:CSD19534Q5A-RESCUE-SB-4S5A Q1
 U 1 1 597E6AFE
 P 5550 1550
@@
 $EndComp
 $Comp
-L CSD19534Q5A Q2
+L SB-4S5A-rescue:CSD19534Q5A-RESCUE-SB-4S5A Q2
 U 1 1 597E6C1E
 P 6550 1550
@@
 $EndComp
 $Comp
-L CONN_01X06 J1
+L Connector:Conn_01x06 J1
 U 1 1 5992673F
-P 9350 4350
-F 0 "J1" H 9268 3875 50  0000 C CNN
-F 1 "CONN_01X06" H 9268 3966 50  0000 C CNN
-F 2 "TI SBS:14110613002XXX" H 9350 4350 50  0001 C CNN
-F 3 "" H 9350 4350 50  0001 C CNN
-	1    9350 4350
+P 9350 4400
+F 0 "J1" H 9268 3925 50  0000 C CNN
+F 1 "CONN_01X06" H 9268 4016 50  0000 C CNN
+F 2 "TI SBS:14110613002XXX" H 9350 4400 50  0001 C CNN
+F 3 "" H 9350 4400 50  0001 C CNN
+	1    9350 4400
 	1    0    0    1
 $EndComp
 $Comp
-L R R20
+L SB-4S5A-rescue:R-RESCUE-SB-4S5A R20
 U 1 1 59926AF9
 P 8600 4500
@@
 $EndComp
 $Comp
-L R R19
+L device:R R19
 U 1 1 59926BB4
 P 8350 4600
@@
 Connection ~ 6650 3400
 $Comp
-L GNDD #PWR01
+L power:GNDD #PWR01
 U 1 1 59980A6F
 P 2650 4700

Commit message: Almost done, can't freaking decide on a connector...
Parts:
- removed J1: CONN_01X06, TI SBS:14110613002XXX, symbol Connector:Conn_01x06
- added J1: Conn_02x03_Top_Bottom, Connectors_Molex:Molex_Microfit3_Header_02x03_Angled_43045-060x, symbol SB-4S5A-rescue:Conn_02x03_Top_Bottom-Connector
- BT1, BT2, BT3, BT4: symbol device:Battery_Cell -> SB-4S5A-rescue:Battery_Cell-device
- C1, C2, C3, C4, C5, C6: symbol device:C -> SB-4S5A-rescue:C-device
- D1: symbol device:D_Schottky -> SB-4S5A-rescue:D_Schottky-device
- Q3: symbol Transistor:2N7002 -> SB-4S5A-rescue:2N7002-Transistor
- R1: footprint Oddities:NetTie-I_Connected -> Resistors_SMD:R_0402
- R17, R19: symbol device:R -> SB-4S5A-rescue:R-device
- TH1, TH2, TH3, TH4: symbol device:Thermistor_NTC -> SB-4S5A-rescue:Thermistor_NTC-device
Connections:
- net BTP_INT: now also J1.6 (Pin_6)
- net PACK+: now also J1.1 (Pin_1)
- net PACK-: now also J1.2 (Pin_2)
- net SMBC: now also J1.3 (Pin_3)
- net SMBD: now also J1.4 (Pin_4)
- net ~PRES~: now also J1.5 (Pin_5)
Changed lines of the file:
@@
 $EndComp
 $Comp
-L device:Battery_Cell BT1
+L SB-4S5A-rescue:Battery_Cell-device BT1
 U 1 1 597D5B15
 P 1650 3000
@@
 $EndComp
 $Comp
-L device:Battery_Cell BT2
+L SB-4S5A-rescue:Battery_Cell-device BT2
 U 1 1 597D5BA3
 P 1650 3500
@@
 $EndComp
 $Comp
-L device:Battery_Cell BT3
+L SB-4S5A-rescue:Battery_Cell-device BT3
 U 1 1 597D5BC7
 P 1650 4000
@@
 $EndComp
 $Comp
-L device:Battery_Cell BT4
+L SB-4S5A-rescue:Battery_Cell-device BT4
 U 1 1 597D5C07
 P 1650 4500
@@
 $EndComp
 $Comp
-L device:D_Schottky D1
+L SB-4S5A-rescue:D_Schottky-device D1
 U 1 1 597D8090
 P 5150 3200
@@
 $EndComp
 $Comp
-L device:R R17
+L SB-4S5A-rescue:R-device R17
 U 1 1 597D94E6
 P 8350 4400
@@
 $EndComp
 $Comp
-L device:C C1
+L SB-4S5A-rescue:C-device C1
 U 1 1 597DA829
 P 2650 2950
@@
 $EndComp
 $Comp
-L device:C C2
+L SB-4S5A-rescue:C-device C2
 U 1 1 597DA9C3
 P 2650 3450
@@
 $EndComp
 $Comp
-L device:C C3
+L SB-4S5A-rescue:C-device C3
 U 1 1 597DAA35
 P 2650 3950
@@
 $EndComp
 $Comp
-L device:C C4
+L SB-4S5A-rescue:C-device C4
 U 1 1 597DAA98
 P 2650 4450
@@
 $EndComp
 $Comp
-L device:Thermistor_NTC TH1
+L SB-4S5A-rescue:Thermistor_NTC-device TH1
 U 1 1 597DB329
 P 4500 4450
@@
 $EndComp
 $Comp
-L device:Thermistor_NTC TH2
+L SB-4S5A-rescue:Thermistor_NTC-device TH2
 U 1 1 597DB805
 P 4650 4450
@@
 $EndComp
 $Comp
-L device:Thermistor_NTC TH3
+L SB-4S5A-rescue:Thermistor_NTC-device TH3
 U 1 1 597DB855
 P 4800 4450
@@
 $EndComp
 $Comp
-L device:Thermistor_NTC TH4
+L SB-4S5A-rescue:Thermistor_NTC-device TH4
 U 1 1 597DB899
 P 4950 4450
@@
 $EndComp
 $Comp
-L device:C C5
+L SB-4S5A-rescue:C-device C5
 U 1 1 597DC7E1
 P 3500 4500
@@
 $EndComp
 Wire Wire Line
-	5850 1350 6250 1350
-Wire Wire Line
-	5850 1450 6250 1450
-Wire Wire Line
-	5850 1550 6250 1550
-Wire Wire Line
-	5850 1650 6250 1650
-Wire Wire Line
-	6050 1350 6050 2150
+	5850 1350 6050 1350
+Wire Wire Line
+	5850 1450 6050 1450
+Wire Wire Line
+	5850 1550 6050 1550
+Wire Wire Line
+	5850 1650 6050 1650
+Wire Wire Line
+	6050 1350 6050 1450
 Connection ~ 6050 1450
 Connection ~ 6050 1350
@@
 	5150 1550 5250 1550
 Wire Wire Line
-	5150 1350 5150 1550
+	5150 1350 5150 1450
 Wire Wire Line
 	5250 1450 5150 1450
@@
 	6950 1550 6850 1550
 Wire Wire Line
-	6950 1350 6950 1550
-Wire Wire Line
-	6850 1350 8250 1350
+	6950 1350 6950 1450
+Wire Wire Line
+	6850 1350 6950 1350
 Wire Wire Line
 	6850 1450 6950 1450
@@
 	6850 1650 7050 1650
 Wire Wire Line
-	7050 1650 7050 2150
+	7050 1650 7050 2050
 Wire Wire Line
 	4800 1350 4800 3200
@@
 	6550 4500 6650 4500
 Wire Wire Line
-	6650 4500 6650 4650
+	6650 4500 6650 4550
 Wire Wire Line
 	6550 4550 6650 4550
@@
 	5550 4450 5450 4450
 Wire Wire Line
-	5450 4450 5450 4650
+	5450 4450 5450 4500
 Wire Wire Line
 	5550 4500 5450 4500
@@
 	8750 4300 9150 4300
 Wire Wire Line
-	8500 4400 9150 4400
-Wire Wire Line
-	1650 4100 1650 4300
-Wire Wire Line
-	1650 3600 1650 3800
-Wire Wire Line
-	1650 3100 1650 3300
-Wire Wire Line
-	1650 1350 1650 2800
+	1650 4100 1650 4200
+Wire Wire Line
+	1650 3600 1650 3700
+Wire Wire Line
+	1650 3100 1650 3200
+Wire Wire Line
+	1650 1350 1650 2700
 Wire Wire Line
 	2100 2700 1650 2700
@@
 Connection ~ 1650 4200
 Wire Wire Line
-	1650 4600 1650 5300
-Wire Wire Line
-	1650 1350 5250 1350
+	1650 4600 1650 4700
+Wire Wire Line
+	1650 1350 4800 1350
 Connection ~ 5150 1350
 Connection ~ 5050 1350
@@
 	3100 2700 3100 3400
 Wire Wire Line
-	2400 2700 3100 2700
+	2400 2700 2650 2700
 Wire Wire Line
 	3050 3450 5550 3450
@@
 	3050 3200 3050 3450
 Wire Wire Line
-	2400 3200 3050 3200
+	2400 3200 2650 3200
 Wire Wire Line
 	3050 3500 5550 3500
@@
 	3050 3700 3050 3500
 Wire Wire Line
-	2400 3700 3050 3700
+	2400 3700 2650 3700
 Wire Wire Line
 	3100 3550 5550 3550
@@
 	3100 4200 3100 3550
 Wire Wire Line
-	2400 4200 3100 4200
+	2400 4200 2650 4200
 Wire Wire Line
 	2650 2700 2650 2800
 Connection ~ 2650 2700
 Wire Wire Line
-	2650 3100 2650 3300
+	2650 3100 2650 3200
 Connection ~ 2650 3200
 Wire Wire Line
-	2650 3600 2650 3800
+	2650 3600 2650 3700
 Connection ~ 2650 3700
 Wire Wire Line
-	2650 4100 2650 4300
+	2650 4100 2650 4200
 Connection ~ 2650 4200
 Wire Wire Line
@@
 	3650 4500 3750 4500
 Wire Wire Line
-	3750 3900 3750 4600
+	3750 3900 3750 4500
 Wire Wire Line
 	3350 4500 3250 4500
 Wire Wire Line
-	3250 3800 3250 4600
+	3250 3800 3250 4500
 Wire Wire Line
 	3650 5100 8250 5100
@@
 $EndComp
 Wire Wire Line
-	4500 4600 4500 4800
-Wire Wire Line
-	4250 4700 4950 4700
+	4500 4600 4500 4700
+Wire Wire Line
+	4250 4700 4500 4700
 Wire Wire Line
 	4950 4700 4950 4600
@@
 $EndComp
 $Comp
-L Transistor:2N7002 Q3
+L SB-4S5A-rescue:2N7002-Transistor Q3
 U 1 1 597DF192
 P 7350 1750
@@
 Connection ~ 7900 1350
 $Comp
-L device:C C6
+L SB-4S5A-rescue:C-device C6
 U 1 1 597E0DFB
 P 4250 4450
@@
 F 0 "R1" V 1900 5300 50  0000 C CNN
 F 1 "NET-TIE" V 1800 5300 50  0000 C CNN
-F 2 "Oddities:NetTie-I_Connected" V 1830 5300 50  0001 C CNN
+F 2 "Resistors_SMD:R_0402" V 1830 5300 50  0001 C CNN
 F 3 "" H 1900 5300 50  0001 C CNN
 	1    1900 5300
@@
 $EndComp
 $Comp
-L Connector:Conn_01x06 J1
-U 1 1 5992673F
-P 9350 4400
-F 0 "J1" H 9268 3925 50  0000 C CNN
-F 1 "CONN_01X06" H 9268 4016 50  0000 C CNN
-F 2 "TI SBS:14110613002XXX" H 9350 4400 50  0001 C CNN
-F 3 "" H 9350 4400 50  0001 C CNN
-	1    9350 4400
-	1    0    0    1
-$EndComp
-$Comp
 L SB-4S5A-rescue:R-RESCUE-SB-4S5A R20
 U 1 1 59926AF9
@@
 $EndComp
 $Comp
-L device:R R19
+L SB-4S5A-rescue:R-device R19
 U 1 1 59926BB4
 P 8350 4600
@@
 	8000 4500 8450 4500
 Wire Wire Line
-	8750 4500 9150 4500
-Wire Wire Line
 	5250 5000 8100 5000
 Wire Wire Line
@@
 Wire Wire Line
 	8100 4600 8200 4600
-Wire Wire Line
-	8500 4600 9150 4600
 Wire Wire Line
 	9150 4100 9000 4100
@@
 Wire Wire Line
 	6850 4300 6550 4300
+Wire Wire Line
+	6050 1450 6250 1450
+Wire Wire Line
+	6050 1450 6050 1550
+Wire Wire Line
+	6050 1350 6250 1350
+Wire Wire Line
+	6050 1550 6250 1550
+Wire Wire Line
+	6050 1550 6050 1650
+Wire Wire Line
+	6050 1650 6250 1650
+Wire Wire Line
+	6050 1650 6050 2150
+Wire Wire Line
+	5150 1450 5150 1550
+Wire Wire Line
+	6950 1450 6950 1550
+Wire Wire Line
+	6950 1350 7050 1350
+Wire Wire Line
+	6650 4550 6650 4650
+Wire Wire Line
+	5450 4500 5450 4550
+Wire Wire Line
+	5450 4550 5450 4650
+Wire Wire Line
+	1650 2700 1650 2800
+Wire Wire Line
+	1650 3200 1650 3300
+Wire Wire Line
+	1650 3700 1650 3800
+Wire Wire Line
+	1650 4200 1650 4300
+Wire Wire Line
+	5150 1350 5250 1350
+Wire Wire Line
+	5050 1350 5150 1350
+Wire Wire Line
+	4800 1350 5050 1350
+Wire Wire Line
+	2650 2700 3100 2700
+Wire Wire Line
+	2650 3200 3050 3200
+Wire Wire Line
+	2650 3200 2650 3300
+Wire Wire Line
+	2650 3700 3050 3700
+Wire Wire Line
+	2650 3700 2650 3800
+Wire Wire Line
+	2650 4200 3100 4200
+Wire Wire Line
+	2650 4200 2650 4300
+Wire Wire Line
+	1650 4700 1650 5300
+Wire Wire Line
+	3250 4500 3250 4600
+Wire Wire Line
+	3750 4500 3750 4600
+Wire Wire Line
+	4650 4700 4800 4700
+Wire Wire Line
+	4800 4700 4950 4700
+Wire Wire Line
+	4500 4700 4500 4800
+Wire Wire Line
+	4500 4700 4650 4700
+Wire Wire Line
+	7250 1350 7900 1350
+Wire Wire Line
+	7050 2050 7050 2150
+Wire Wire Line
+	7900 1350 8250 1350
+Wire Wire Line
+	7050 1350 7250 1350
+$Comp
+L SB-4S5A-rescue:Conn_02x03_Top_Bottom-Connector J1
+U 1 1 5A5A1977
+P 9350 4200
+F 0 "J1" H 9400 4517 50  0000 C CNN
+F 1 "Conn_02x03_Top_Bottom" H 9400 4426 50  0000 C CNN
+F 2 "Connectors_Molex:Molex_Microfit3_Header_02x03_Angled_43045-060x" H 9350 4200 50  0001 C CNN
+F 3 "~" H 9350 4200 50  0001 C CNN
+	1    9350 4200
+	1    0    0    -1
+$EndComp
+Wire Wire Line
+	9850 4200 9650 4200
+Wire Wire Line
+	8750 4500 9850 4500
+Wire Wire Line
+	9650 4100 9950 4100
+Wire Wire Line
+	9950 4400 9950 4100
+Wire Wire Line
+	8500 4400 9950 4400
+Wire Wire Line
+	9850 4500 9850 4200
+Wire Wire Line
+	10050 4300 10050 4600
+Wire Wire Line
+	9650 4300 10050 4300
+Wire Wire Line
+	8500 4600 10050 4600
 $EndSCHEMATC

Commit message: Ready to send to manufacturer.
Parts:
- removed J1: Conn_02x03_Top_Bottom, Connectors_Molex:Molex_Microfit3_Header_02x03_Angled_43045-060x, symbol SB-4S5A-rescue:Conn_02x03_Top_Bottom-Connector
- added J1: LEMO6, Connectors_Samtec:SL-106-X-XX_1x06, symbol Connector_Specialized:LEMO6
Connections:
- wire segments 183 -> 187
Changed lines of the file:
@@
 	8100 4600 8200 4600
 Wire Wire Line
-	9150 4100 9000 4100
-Wire Wire Line
-	9000 4100 9000 3700
+	9150 3600 9000 3600
+Wire Wire Line
+	9000 3600 9000 3700
 Wire Wire Line
 	9000 3700 8600 3700
@@
 PACK-
 Wire Wire Line
-	9150 4200 8900 4200
-Wire Wire Line
-	8900 4200 8900 3850
+	9650 3900 8900 3900
+Wire Wire Line
+	8900 3900 8900 3850
 Wire Wire Line
 	8900 3850 8600 3850
@@
 Wire Wire Line
 	7050 1350 7250 1350
+Wire Wire Line
+	9150 2800 10450 2800
+Wire Wire Line
+	8500 4400 10250 4400
 $Comp
-L SB-4S5A-rescue:Conn_02x03_Top_Bottom-Connector J1
-U 1 1 5A5A1977
-P 9350 4200
-F 0 "J1" H 9400 4517 50  0000 C CNN
-F 1 "Conn_02x03_Top_Bottom" H 9400 4426 50  0000 C CNN
-F 2 "Connectors_Molex:Molex_Microfit3_Header_02x03_Angled_43045-060x" H 9350 4200 50  0001 C CNN
-F 3 "~" H 9350 4200 50  0001 C CNN
-	1    9350 4200
+L Connector_Specialized:LEMO6 J1
+U 1 1 5AC3E2DD
+P 9650 3400
+F 0 "J1" H 9650 4078 50  0000 C CNN
+F 1 "LEMO6" H 9650 3987 50  0000 C CNN
+F 2 "Connectors_Samtec:SL-106-X-XX_1x06" H 9650 3400 50  0001 C CNN
+F 3 "" H 9650 3400 50  0001 C CNN
+	1    9650 3400
 	1    0    0    -1
 $EndComp
 Wire Wire Line
-	9850 4200 9650 4200
-Wire Wire Line
-	8750 4500 9850 4500
-Wire Wire Line
-	9650 4100 9950 4100
-Wire Wire Line
-	9950 4400 9950 4100
-Wire Wire Line
-	8500 4400 9950 4400
-Wire Wire Line
-	9850 4500 9850 4200
-Wire Wire Line
-	10050 4300 10050 4600
-Wire Wire Line
-	9650 4300 10050 4300
-Wire Wire Line
-	8500 4600 10050 4600
+	9150 4300 9150 4000
+Wire Wire Line
+	9150 4000 10150 4000
+Wire Wire Line
+	10150 4000 10150 3600
+Wire Wire Line
+	10150 3200 10250 3200
+Wire Wire Line
+	8750 4500 10350 4500
+Wire Wire Line
+	9650 2900 10350 2900
+Wire Wire Line
+	9150 2800 9150 3200
+Wire Wire Line
+	10250 4400 10250 3200
+Wire Wire Line
+	10350 4500 10350 2900
+Wire Wire Line
+	10450 4600 10450 2800
+Wire Wire Line
+	8500 4600 10450 4600
 $EndSCHEMATC
